File: Hardware/Production/RTK_Control-Panel.brd (EAGLE design)
At the start: 151.8 x 101.6 mm, 406 parts, among them J3 MICRO-SD-PUSH-PUSH-EXT-PIN, J4 Vertical Qwiic Connector, J9 MAGJACK-POE, U1 ESP32-WROVER-IE, U10 POE_PSU-DP990X, U11 MCP6021T, U12 AP7361C-33, U13 MCP6021T, U14 BP2G1+_POWER_SPLITTER, U15 USB251XB, U16 SN74AVC4T774PW, U17 URB2405YMD-15WR3, U2 CH340C, U3 XC6222B331MR-G, U4 U-BLOX_ZED-F9P, U5 U-BLOX_NEO-D9S-00B, U6 XC6222B331MR-G, U7 W5500, U8 LARA-R6001, U9 74LVC4066D_QUAD_BILATERAL_SWI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, Y1 25MHz, Y2 24MHz

Commit message: Ready for Proto Review
Parts:
- removed FRAME1: FRAME-LEDGER, SparkFun-Aesthetics:CREATIVE_COMMONS
- removed FRAME2: FRAME-LEDGERNO_FOOTPRINT, SparkFun-Aesthetics:DUMMY
- removed LOGO1: SPECIAL_INSTRUCTIONS-ORDERING, SparkFun-Aesthetics:ORDERING_INSTRUCTIONS
- added E$1, E$2, E$3, E$4: (no value), SparkFun-Aesthetics:FIDUCIAL-1X2
- added E$5, E$6: (no value), SparkFun-Retired:FIDUCIAL-1.5X3
- moved C68 0.32 mm to (131.8, 16.5)
- moved H1 0.32 mm to (149.5, 2.54)
- moved H2 0.32 mm to (149.5, 99.1)
- moved JP2 0.32 mm to (134.0, 19.1)
- moved R67 0.32 mm to (129.9, 30.5)
- moved U8 0.32 mm to (131.8, 72.4)
- moved !SAFEBOOT_ZED! 0.32 mm to (106.4, 87.6)
- moved ANT_DET 0.32 mm to (70.8, 38.1)
- moved ANT_SHT 0.32 mm to (70.8, 48.3)
- moved C12 0.32 mm to (95.6, 72.4)
- moved C13 0.32 mm to (97.5, 90.8)
- moved C2 0.32 mm to (84.0, 30.5)
- moved C25 0.32 mm to (68.9, 22.9)
- moved C3 0.32 mm to (109.2, 27.1)
- moved C4 0.32 mm to (109.2, 25.4)
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Other:
- board size 151.8 x 101.6 mm -> 171.8 x 115.8 mm
- board text added: "v-score"
- board text removed: "Dimensions In Inches"
- board text removed: "JLCPCB JLC-7628 Impedance Control 4-Layers Thickness: 1.6mm Outer Copper: 1oz Finish: HASL Lead Free Red Solder Resist White Silkscreen"
- board text removed: "Paul Clark"
- board text removed: "V-Score To V-Score"
