File: Hardware/Production/RTK_Everywhere_L-Band_Cellular-Panel.brd (EAGLE design)
At the start: 171.8 x 115.8 mm, 409 parts, among them J3 MICRO-SD-PUSH-PUSH-EXT-PIN, J4 Vertical Qwiic Connector, J9 MAGJACK-POE, U1 ESP32-WROVER-IE, U10 POE_PSU-DP990X, U11 MCP6021T, U12 AP7361C-33, U13 MCP6021T, U14 BP2G1+_POWER_SPLITTER, U15 USB251XB_USB2514B, U16 SN74AVC4T774PW, U17 URB2405YMD, U2 CH340C, U3 XC6222B331MR-G, U4 U-BLOX_ZED-F9P, U5 U-BLOX_NEO-D9S-00B, U6 XC6222B331MR-G, U7 W5500, U8 LARA-R6001D, U9 74LVC4066D_QUAD_BILATERAL_SWI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, Y1 25MHz, Y2 24MHz

Commit message: Add no L-Band bypass. Update silk. Increase display cutout.
Parts:
- added JPP1, JPP2: NO PASTE, SparkFun-Jumpers:SMT-JUMPER_2_SOIC-PAD_NO-PASTE
- added U$2, U$90: (no value), output:RTK_EVERYWHERE0
- added U$91, U$92: (no value), output:NO0
- added U$96: (no value), output:CELLULAR2
- added U$97: (no value), output:L#BAND1
- moved LOGO4 39.6 mm to (121.6, 30.5)
- moved E$5 5.08 mm to (6.86, -7.18)
- moved E$6 5.08 mm to (6.86, -7.18)
- moved E$1 5.08 mm to (6.86, 108.8)
- moved E$2 5.08 mm to (6.86, 108.8)
- moved E$3 5.08 mm to (144.8, 108.8)
- moved E$4 5.08 mm to (144.8, 108.8)
- moved LOGO6 2.84 mm to (125.2, 44.5)
- moved U$152 2.84 mm to (138.1, 41.4)
- moved LOGO5 2.84 mm to (121.6, 39.4)
- moved J13 0.63 mm to (46.7, 98.4)
Connections:
- net N$42 renamed ANT
- new net BYPASS: JPP1.1, JPP2.1
Routing:
- net BYPASS: track 0.00 -> 3.47 mm
- net VIN-: track 6.29 -> 6.93 mm
- net VIN+: track 5.90 -> 6.53 mm
- net 3.3V_SW: track 146.4 -> 147.1 mm
Other:
- board size 171.8 x 115.8 mm -> 165.5 x 131.1 mm
- board text added: "Route Out"

Commit message: Update RF Bypass SOIC Pad jumpers
Parts:
- removed JPP1, JPP2: NO PASTE, SparkFun-Jumpers:SMT-JUMPER_2_SOIC-PAD_NO-PASTE
- added BYPASS1, BYPASS2: NO PASTE, SparkFun-Jumpers:SMT-JUMPER_2_SOIC-PAD_NO-PASTE
Connections:
- net BYPASS: now also BYPASS1.1, BYPASS2.1; no longer JPP1.1, JPP2.1
Routing:
- net BYPASS: track 3.47 -> 4.03 mm
Changed lines of the file:
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@@
 <element name="U$79" library="output" package="UART14" value="" x="74.6125" y="72.898" smashed="yes" rot="MR0"/>
 <element name="U$89" library="output" package="4_#_#SD_CS#15" value="" x="50.4825" y="10.922" smashed="yes" rot="MR270"/>
-<element name="JPP1" library="SparkFun-Jumpers" package="SMT-JUMPER_2_SOIC-PAD_NO-PASTE" value="NO PASTE" x="97.4725" y="86.487" smashed="yes" rot="R90"/>
-<element name="JPP2" library="SparkFun-Jumpers" package="SMT-JUMPER_2_SOIC-PAD_NO-PASTE" value="NO PASTE" x="98.7425" y="83.693" smashed="yes" rot="R270"/>
+<element name="BYPASS1" library="SparkFun-Jumpers" package="SMT-JUMPER_2_SOIC-PAD_NO-PASTE" value="NO PASTE" x="97.4725" y="85.09" smashed="yes" rot="R90">
+<attribute name="VALUE" value="NO PASTE" x="97.4725" y="85.09" size="1.778" layer="27" rot="R90" display="off"/>
+</element>
+<element name="BYPASS2" library="SparkFun-Jumpers" package="SMT-JUMPER_2_SOIC-PAD_NO-PASTE" value="NO PASTE" x="98.7425" y="85.09" smashed="yes" rot="R270">
+<attribute name="VALUE" value="NO PASTE" x="98.7425" y="85.09" size="1.778" layer="27" rot="R270" display="off"/>
+</element>
 <element name="U$2" library="output" package="RTK_EVERYWHERE0" value="" x="126.6825" y="35.56" smashed="yes"/>
 <element name="U$90" library="output" package="RTK_EVERYWHERE0" value="" x="119.0625" y="45.72" smashed="yes" rot="MR0"/>
@@
 </signal>
 <signal name="BYPASS">
-<contactref element="JPP1" pad="1"/>
-<contactref element="JPP2" pad="1"/>
-<wire x1="97.4725" y1="86.487" x2="97.4725" y2="85.598" width="0.348996875" layer="1"/>
-<wire x1="97.4725" y1="85.598" x2="97.9805" y2="85.09" width="0.348996875" layer="1" curve="90"/>
-<wire x1="97.9805" y1="85.09" x2="98.2345" y2="85.09" width="0.348996875" layer="1"/>
-<wire x1="98.2345" y1="85.09" x2="98.7425" y2="84.582" width="0.348996875" layer="1" curve="-90"/>
-<wire x1="98.7425" y1="84.582" x2="98.7425" y2="83.693" width="0.348996875" layer="1"/>
+<contactref element="BYPASS1" pad="1"/>
+<contactref element="BYPASS2" pad="1"/>
+<wire x1="97.4725" y1="86.84" x2="97.4725" y2="85.725" width="0.348996875" layer="1"/>
+<wire x1="97.4725" y1="85.725" x2="98.1075" y2="85.09" width="0.348996875" layer="1" curve="90"/>
+<wire x1="98.1075" y1="85.09" x2="98.7425" y2="84.455" width="0.348996875" layer="1" curve="-90"/>
+<wire x1="98.7425" y1="84.455" x2="98.7425" y2="83.34" width="0.348996875" layer="1"/>
 </signal>
 </signals>

Commit message: Add V10 PCB files
Parts:
- removed Q3, Q4: (no value), SparkFun-DiscreteSemi:SC70-6
- removed R69: 10k, SparkFun-Resistors:0603
- added D15, D16, D17, D18, D19, D20: PESD0402-0402, SparkFun-DiscreteSemi:0402
- added Q5, Q6: 310mA/60V/1.6Ω, SparkFun-DiscreteSemi:SOT323
- added R50, R51, R52: 100k, SparkFun-Resistors:0603
- added RXD, TXD, VCCIO: TEST-POINTPOGO_PTH, SparkFun-Connectors:1X01_NO_SILK
- added SPWR, TPWR: JUMPER-SMT_3_1-NC_TRACE_SILK, SparkFun-Jumpers:SMT-JUMPER_3_1-NC_TRACE_SILK
- added U$103: (no value), output:13_#_TXDI15
- added U$108: (no value), output:14_#_RXDO0
- added U$110, U$112: (no value), output:LARA_ON0
- added U$115, U$116: (no value), output:VCCIO0
- added U$117: (no value), output:#3V3_SW_EN#0
- added U$118: (no value), output:#3V3_SW2_EN#0
- added U18: 74HC1G04, SparkFun-IC-Logic:SOT353
- R44: value 10k -> 100k
- U$73: device output:50 -> output:14_#_RXDO0
- U$75: device output:50 -> output:13_#_TXDI15
- moved R44 37.6 mm to (126.8, 16.5), turned to 90 degrees
- moved U$75 32.3 mm to (111.8, 29.2), flipped to the top
- moved U$73 31.9 mm to (111.3, 31.8)
- moved LOGO7 22.5 mm to (130.5, 71.1)
- moved LOGO8 22.5 mm to (126.9, 76.2)
- moved U$90 22.5 mm to (125.4, 67.3)
- moved U$153 22.5 mm to (114.0, 73.3)
- moved E$5 16.5 mm to (-2.62, 6.35)
- moved E$6 16.5 mm to (-2.62, 6.35)
- moved E$3 10.7 mm to (154.4, 104.0)
- moved E$4 10.7 mm to (154.4, 104.0)
- moved E$1 10.6 mm to (-2.62, 104.0)
- moved E$2 10.6 mm to (-2.62, 104.0)
- moved U$48 3.56 mm to (133.0, 17.2)
- moved U$135 3.43 mm to (46.7, 30.1)
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- renumbered ESP5 to LARA_ON, JP1 to USB251SDA, JP2 to USB251SCL
Connections:
- net ESP26/LARA_ON renamed ESP26/LARA_PWR_ON
- net ESP5 renamed ESP5/LARA_ON
- removed net N$37: LARA_ON.1, U9.9
- removed net N$57: U15.22, USB251SDA.2
- removed net N$58: U15.24, USB251SCL.2
- removed net N$59: Q4.2, Q4.3, R69.1
- removed net N$60: Q3.5, R68.2
- new net LARA_ON: LARA_ON.1, U16.11, U9.9
- new net N$22: R50.1, SPWR.3
- new net N$26: SPWR.2, U3.3
- new net N$31: R51.1, TPWR.3
- new net N$39: TPWR.2, U12.5
- new net N$42: Q6.1, R68.2
- new net USB251SCL: R52.2, U15.24, USB251SCL.2
- new net USB251SDA: R44.2, U15.22, USB251SDA.2
- net 3.3V_SW2: now also U18.5; no longer R44.2, R69.2
- net 5V: now also R50.2, R51.2
- net ESP13/LARA_TXDI: now also TXD.1
- net ESP14/LARA_RXDO: now also RXD.1
- net ESP21/SDA: now also D15.1
- net ESP22/SCL: now also D16.1
- net ESP25/TP: now also D20.1
- net GND: now also D15.2, D16.2, D17.2, D18.2, D19.2, D20.2, Q5.2, Q6.2, R44.1, R52.1, U18.3; no longer Q3.1, Q3.4, Q4.1, Q4.4
- net GNSS_!RESET!: now also U18.2; no longer R68.1
- net LARA_!RESET!: now also Q6.3; no longer Q3.6
- net LARA_PWR_ON: now also Q5.3; no longer Q4.6
- net N$16: now also R68.1, U18.4; no longer Q3.2, Q3.3, R44.1
- net N$65: now also Q5.1; no longer Q4.5
- net PWREN: now also SPWR.1, TPWR.1; no longer U12.5, U3.3
- net VCCIO: now also VCCIO.1
- net ZED_EXTINT: now also D19.1
- net ZED_RX2: now also D17.1
- net ZED_TX2: now also D18.1
Routing:
- net LARA_ON: track 0.00 -> 59.5 mm, vias 0 -> 1
- net N$31: track 0.00 -> 17.5 mm, vias 0 -> 1
- net N$22: track 0.00 -> 9.95 mm, vias 0 -> 1
- net USB251SDA: track 0.00 -> 9.37 mm, vias 0 -> 1
- net USB251SCL: track 0.00 -> 9.24 mm, vias 0 -> 1
- net ESP13/LARA_TXDI: track 29.8 -> 38.8 mm
- net ESP14/LARA_RXDO: track 34.1 -> 40.3 mm
- net LARA_!RESET!: track 19.1 -> 14.1 mm
- net VCCIO: track 52.0 -> 57.0 mm
- net N$59: track 4.65 -> 0.00 mm
- net ESP0/!BOOT!: track 67.1 -> 70.7 mm
- net RD-: track 28.9 -> 32.1 mm
- net N$37: track 3.07 -> 0.00 mm
- net N$26: track 0.00 -> 3.03 mm, vias 0 -> 1
- net N$39: track 0.00 -> 2.84 mm, vias 0 -> 1
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- added copper zone on layer 15, net 3.3_SW
Other:
- board text added: "v10"
- board text removed: "v01"
