File: Hardware/Production/SparkFun_RTK_EVK-Panel.brd (EAGLE design)
At the start: 151.8 x 101.6 mm, 437 parts, among them J3 MICRO-SD-PUSH-PUSH-EXT-PIN, J4 Vertical Qwiic Connector, J9 MAGJACK-POE, Q5 310mA/60V/1.6Ω, Q6 310mA/60V/1.6Ω, U1 ESP32-WROVER-IE, U10 POE_PSU-DP990X, U11 MCP6021T, U12 AP7361C-33, U13 MCP6021T, U14 BP2G1+_POWER_SPLITTER, U15 USB251XB_USB2514B, U16 SN74AVC4T774PW, U17 URB2405YMD, U18 74HC1G04, U2 CH340C, U3 XC6222B331MR-G, U4 U-BLOX_ZED-F9P, U5 U-BLOX_NEO-D9S-00B, U6 XC6222B331MR-G, U7 W5500, U8 LARA-R6001D, U9 74LVC4066D_QUAD_BILATERAL_SWI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, Y1 25MHz, Y2 24MHz

Commit message: v11 PCB
Parts:
- removed FRAME1: FRAME-LEDGER, SparkFun-Aesthetics:CREATIVE_COMMONS
- removed FRAME2: FRAME-LEDGERNO_FOOTPRINT, SparkFun-Aesthetics:DUMMY
- removed LARA_ON: TEST-POINTPOGO_PTH, SparkFun-Connectors:1X01_NO_SILK
- removed LOGO1: SPECIAL_INSTRUCTIONS-ORDERING, SparkFun-Aesthetics:ORDERING_INSTRUCTIONS
- removed RX-TX, TX-RX: JUMPER-COMBO_2_NC_TRACE, SparkFun-Jumpers:COMBO-JUMPER_2_NC_TRACE
- removed U$109, U$27: (no value), output:33_#_#ETH_INT#0
- removed U$112: (no value), output:LARA_ON0
- added E$1, E$2, E$3, E$4: (no value), SparkFun-Aesthetics:FIDUCIAL-1X2
- added E$5, E$6: (no value), SparkFun-Retired:FIDUCIAL-1.5X3
- added NEO_RX, NEO_TX, ZED_RXI, ZED_TXO: TEST-POINTPOGO_PTH, SparkFun-Connectors:1X01_NO_SILK
- U$11: device output:ZED_TX1 -> output:RTK_EVK0
- U$110: device output:LARA_ON0 -> output:39_#_#ETH_INT#0
- U$13: device output:ZED_RX0 -> output:RTK_EVK0
- U$2: device output:RTK_EVERYWHERE0 -> output:33_#_ZED_RXI0
- U$79: device output:UART14 -> output:39_#_#ETH_INT#0
- U$90: device output:RTK_EVERYWHERE0 -> output:25_#_ZED_TXO0
- moved U$11 63.5 mm to (124.1, 35.6), flipped to the top
- moved U$13 60.8 mm to (130.5, 67.3)
- moved U$79 49.0 mm to (99.0, 30.2), flipped to the top
- moved U$90 28.2 mm to (111.1, 43.2)
- moved U$2 21.1 mm to (111.1, 45.7), flipped to the bottom
- moved U$110 16.0 mm to (97.2, 31.9), flipped to the bottom
- moved C68 0.32 mm to (131.8, 16.5)
- moved H1 0.32 mm to (149.5, 2.54)
- moved H2 0.32 mm to (149.5, 99.1)
- moved R67 0.32 mm to (129.9, 30.5)
- moved R70 0.32 mm to (131.8, 49.5)
- moved U$92 0.32 mm to (131.8, 73.7)
- moved U$96 0.32 mm to (131.8, 71.1)
- moved U8 0.32 mm to (131.8, 72.4)
- moved USB251SCL 0.32 mm to (134.0, 19.1)
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Connections:
- net ESP5/LARA_ON renamed ESP5/TP
- removed net ESP25/TP: D20.1, J13.1, R6.2, TP.1, U1.10
- removed net ESP33/!ETH_INT!: ETH_INT.1, U1.9, U7.36
- removed net LARA_ON: LARA_ON.1, U16.11, U9.9
- removed net ZED_RXI: RX-TX.2, RX-TX.4, U4.43
- removed net ZED_TXO: TX-RX.1, TX-RX.3, U4.42
- new net ESP25/ZED_TXO: U1.10, U4.42, ZED_TXO.1
- new net ESP33/ZED_RXI: U1.9, U4.43, ZED_RXI.1
- new net ESP39/!ETH_INT!: ETH_INT.1, U1.5, U7.36
- new net ZED_TP: D20.1, J13.1, R6.2, TP.1, U9.9
- net NEO_RXI: now also NEO_RX.1; no longer TX-RX.2, TX-RX.4
- net NEO_TXO: now also NEO_TX.1; no longer RX-TX.1, RX-TX.3
Routing:
- net ESP25/TP: track 141.9 -> 0.00 mm, vias 5 -> 0
- net ZED_TP: track 0.00 -> 135.9 mm, vias 0 -> 3
- net ESP39/!ETH_INT!: track 0.00 -> 96.8 mm, vias 0 -> 4
- net ESP33/!ETH_INT!: track 95.2 -> 0.00 mm, vias 4 -> 0
- net ESP25/ZED_TXO: track 0.00 -> 90.9 mm, vias 0 -> 4
- net ESP33/ZED_RXI: track 0.00 -> 89.2 mm, vias 0 -> 4
- net ZED_RXI: track 84.0 -> 0.00 mm, vias 1 -> 0
- net ZED_TXO: track 77.4 -> 0.00 mm, vias 1 -> 0
- net LARA_ON: track 59.5 -> 0.00 mm, vias 1 -> 0
- net ESP5/TP: track 41.6 -> 36.7 mm, vias 2 -> 0
- net RD-: track 32.1 -> 36.1 mm
- net ESP0/!BOOT!: track 70.7 -> 67.3 mm
- net RXN1: track 17.2 -> 20.0 mm, vias 0 -> 3
- net VCCA: track 69.6 -> 72.3 mm
- net CH340-RXI: track 52.4 -> 49.7 mm
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Other:
- board size 151.8 x 101.6 mm -> 165.5 x 131.1 mm
- board text added: "Route Out"
- board text added: "v-score"
- board text added: "v11"
- board text removed: "Controlled Impedance: JLC7628 Material: TG155 4-Layers Thickness: 1.6mm Outer Copper: 1oz Inner Copper: 0.5oz Finish: HASL Lead Free Red Solder Resist White Silkscreen"
- board text removed: "Dimensions In Inches"
- board text removed: "Paul Clark"
- board text removed: "V-Score To V-Score"
- board text removed: "v10"

Commit message: Final tweaks
Parts:
- I2C: value JUMPER-SMT_3_2-NC_TRACE_SILK -> JUMPER-SMT_3_NO_SILK; device SparkFun-Jumpers:SMT-JUMPER_3_2-NC_TRACE_SILK -> SparkFun-Jumpers:SMT-JUMPER_3_NO_SILK
- moved NEO_RX 2.54 mm to (73.3, 68.6)
- moved NEO_TX 2.54 mm to (73.3, 71.1)
- moved U$14 2.54 mm to (77.2, 71.1)
- moved U$15 2.54 mm to (77.2, 68.6)
- moved U$152 1.80 mm to (139.4, 40.1)
- moved U$153 1.80 mm to (115.3, 72.0)
Routing:
- net NEO_RXI: track 4.73 -> 7.27 mm
- net NEO_TXO: track 4.18 -> 6.72 mm
Changed lines of the file:
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@@
 <attribute name="VALUE" x="69.9865" y="22.86" size="0.6096" layer="27" font="vector" ratio="20" rot="R270" align="top-center"/>
 </element>
-<element name="I2C" library="SparkFun-Jumpers" package="SMT-JUMPER_3_2-NC_TRACE_SILK" package3d_urn="urn:adsk.eagle:package:39289/1" value="JUMPER-SMT_3_2-NC_TRACE_SILK" x="75.8825" y="15.24" smashed="yes" rot="MR0">
+<element name="I2C" library="SparkFun-Jumpers" package="SMT-JUMPER_3_NO_SILK" package3d_urn="urn:adsk.eagle:package:39285/1" value="JUMPER-SMT_3_NO_SILK" x="75.8825" y="15.24" smashed="yes" rot="MR0">
 <attribute name="NAME" x="75.8825" y="16.383" size="0.6096" layer="26" font="vector" ratio="20" rot="MR0" align="bottom-center"/>
 </element>
@@
 <attribute name="VALUE" x="82.1055" y="16.51" size="0.6096" layer="27" font="vector" ratio="20" rot="R90" align="top-center"/>
 </element>
-<element name="U$152" library="output" package="RTK5#SVG0" value="" x="140.6525" y="41.402" smashed="yes"/>
-<element name="U$153" library="output" package="RTK5#SVG0" value="" x="113.9825" y="73.279" smashed="yes" rot="MR0"/>
+<element name="U$152" library="output" package="RTK5#SVG0" value="" x="139.3825" y="40.132" smashed="yes"/>
+<element name="U$153" library="output" package="RTK5#SVG0" value="" x="115.2525" y="72.009" smashed="yes" rot="MR0"/>
 <element name="J13" library="SparkFun-Connectors" package="1X10_SCREW_TERMINAL_3.5MM" value="" x="46.6725" y="98.425" smashed="yes" rot="R180">
 <attribute name="NAME" x="46.6725" y="93.345" size="1.27" layer="25" rot="R180" align="bottom-center"/>
@@
 <element name="U$71" library="output" package="VIN#1" value="" x="34.3535" y="88.773" smashed="yes" rot="MR270"/>
 <element name="U$72" library="output" package="VIN#1" value="" x="34.3535" y="88.9" smashed="yes" rot="R90"/>
-<element name="U$14" library="output" package="NEO_TX2" value="" x="79.6925" y="71.12" smashed="yes" rot="MR0"/>
-<element name="U$15" library="output" package="NEO_RX3" value="" x="79.6925" y="68.58" smashed="yes" rot="MR0"/>
+<element name="U$14" library="output" package="NEO_TX2" value="" x="77.1525" y="71.12" smashed="yes" rot="MR0"/>
+<element name="U$15" library="output" package="NEO_RX3" value="" x="77.1525" y="68.58" smashed="yes" rot="MR0"/>
 <element name="U$89" library="output" package="4_#_#SD_CS#15" value="" x="50.4825" y="10.922" smashed="yes" rot="MR270"/>
 <element name="BYPASS1" library="SparkFun-Jumpers" package="SMT-JUMPER_2_SOIC-PAD_NO-PASTE" value="NO PASTE" x="97.4725" y="85.09" smashed="yes" rot="R90">
@@
 <attribute name="VALUE" x="132.6515" y="49.53" size="0.6096" layer="27" font="vector" ratio="20" rot="R270" align="top-center"/>
 </element>
-<element name="NEO_TX" library="SparkFun-Connectors" package="1X01_NO_SILK" value="TEST-POINTPOGO_PTH" x="75.8825" y="71.12" smashed="yes">
-<attribute name="NAME" x="74.6125" y="72.263" size="0.6096" layer="25" font="vector" ratio="20"/>
-<attribute name="VALUE" x="74.6125" y="69.342" size="0.6096" layer="27" font="vector" ratio="20"/>
-</element>
-<element name="NEO_RX" library="SparkFun-Connectors" package="1X01_NO_SILK" value="TEST-POINTPOGO_PTH" x="75.8825" y="68.58" smashed="yes">
-<attribute name="NAME" x="74.6125" y="69.723" size="0.6096" layer="25" font="vector" ratio="20"/>
-<attribute name="VALUE" x="74.6125" y="66.802" size="0.6096" layer="27" font="vector" ratio="20"/>
+<element name="NEO_TX" library="SparkFun-Connectors" package="1X01_NO_SILK" value="TEST-POINTPOGO_PTH" x="73.3425" y="71.12" smashed="yes">
+<attribute name="NAME" x="72.0725" y="72.263" size="0.6096" layer="25" font="vector" ratio="20"/>
+<attribute name="VALUE" x="72.0725" y="69.342" size="0.6096" layer="27" font="vector" ratio="20"/>
+</element>
+<element name="NEO_RX" library="SparkFun-Connectors" package="1X01_NO_SILK" value="TEST-POINTPOGO_PTH" x="73.3425" y="68.58" smashed="yes">
+<attribute name="NAME" x="72.0725" y="69.723" size="0.6096" layer="25" font="vector" ratio="20"/>
+<attribute name="VALUE" x="72.0725" y="66.802" size="0.6096" layer="27" font="vector" ratio="20"/>
 </element>
 <element name="ZED_TXO" library="SparkFun-Connectors" package="1X01_NO_SILK" value="TEST-POINTPOGO_PTH" x="111.4425" y="43.18" smashed="yes">
@@
 <vertex x="53.0225" y="68.199"/>
 <vertex x="29.4005" y="68.199"/>
-<vertex x="13.6525" y="83.947"/>
+<vertex x="14.9225" y="82.677"/>
+<vertex x="14.9225" y="84.201"/>
+<vertex x="13.6525" y="85.414971875"/>
 </polygon>
 <wire x1="145.8595" y1="100.33" x2="145.8595" y2="99.314" width="0" layer="19" extent="1-1"/>
@@
 <wire x1="47.9785" y1="72.68" x2="47.9425" y2="72.644" width="0.254" layer="1"/>
 <via x="47.9425" y="72.644" extent="1-16" drill="0.3"/>
-<wire x1="55.5625" y1="69.596" x2="53.5305" y2="69.596" width="0.8128" layer="15"/>
-<wire x1="53.5305" y1="69.596" x2="52.5145" y2="69.596" width="0.8128" layer="15"/>
-<wire x1="52.5145" y1="69.596" x2="48.1965" y2="69.596" width="0.8128" layer="15"/>
-<wire x1="47.9425" y1="69.85" x2="48.1965" y2="69.596" width="0.8128" layer="15"/>
 <via x="55.5625" y="69.596" extent="1-16" drill="0.3"/>
 <wire x1="55.5625" y1="69.596" x2="55.5425" y2="69.616" width="0.254" layer="1"/>
@@
 <wire x1="47.9425" y1="72.644" x2="47.9425" y2="69.85" width="0.6096" layer="2"/>
 <wire x1="40.3225" y1="79.375" x2="40.3225" y2="82.55" width="0.6096" layer="2"/>
+<wire x1="47.9425" y1="69.85" x2="48.1965" y2="69.596" width="0.6096" layer="2"/>
+<wire x1="48.1965" y1="69.596" x2="52.5145" y2="69.596" width="0.6096" layer="2"/>
+<wire x1="52.5145" y1="69.596" x2="53.5305" y2="69.596" width="0.6096" layer="2"/>
+<wire x1="53.5305" y1="69.596" x2="55.5625" y2="69.596" width="0.6096" layer="2"/>
 </signal>
 <signal name="N$23">
@@
 <via x="70.8025" y="16.383" extent="1-16" drill="0.3"/>
 <wire x1="70.8025" y1="16.383" x2="71.4375" y2="17.018" width="0.1524" layer="16"/>
-<wire x1="74.8411" y1="16.4084" x2="74.8411" y2="15.24" width="0.1524" layer="16"/>
 <wire x1="71.4375" y1="17.018" x2="74.2315" y2="17.018" width="0.1524" layer="16"/>
-<wire x1="74.2315" y1="17.018" x2="74.8411" y2="16.4084" width="0.1524" layer="16"/>
+<wire x1="75.0697" y1="16.1798" x2="75.0697" y2="15.24" width="0.1524" layer="16"/>
+<wire x1="74.2315" y1="17.018" x2="75.0697" y2="16.1798" width="0.1524" layer="16"/>
 </signal>
 <signal name="N$15">
@@
 <via x="78.4225" y="16.4235" extent="1-16" drill="0.3"/>
 <wire x1="78.4225" y1="16.4235" x2="78.4225" y2="15.748" width="0.1524" layer="16"/>
-<wire x1="77.9145" y1="15.24" x2="76.9239" y2="15.24" width="0.1524" layer="16"/>
+<wire x1="77.9145" y1="15.24" x2="76.6953" y2="15.24" width="0.1524" layer="16"/>
 <wire x1="78.4225" y1="15.748" x2="77.9145" y2="15.24" width="0.1524" layer="16"/>
 </signal>
@@
 <contactref element="U5" pad="20"/>
 <contactref element="NEO_TX" pad="1"/>
-<wire x1="80.0425" y1="71.06" x2="75.9425" y2="71.06" width="0.1524" layer="1"/>
-<wire x1="75.9425" y1="71.06" x2="75.8825" y2="71.12" width="0.1524" layer="1"/>
+<wire x1="80.0425" y1="71.06" x2="73.4025" y2="71.06" width="0.1524" layer="1"/>
+<wire x1="73.4025" y1="71.06" x2="73.3425" y2="71.12" width="0.1524" layer="1"/>
 </signal>
 <signal name="NEO_RXI">
 <contactref element="U5" pad="21"/>
 <contactref element="NEO_RX" pad="1"/>
-<wire x1="80.0425" y1="69.96" x2="77.2625" y2="69.96" width="0.1524" layer="1"/>
-<wire x1="77.2625" y1="69.96" x2="75.8825" y2="68.58" width="0.1524" layer="1"/>
+<wire x1="80.0425" y1="69.96" x2="74.7225" y2="69.96" width="0.1524" layer="1"/>
+<wire x1="74.7225" y1="69.96" x2="73.3425" y2="68.58" width="0.1524" layer="1"/>
 </signal>
 <signal name="N$46">
