File: Hardware/RTK_Control.brd (EAGLE design)
At the start: 151.8 x 101.6 mm, 406 parts, among them J3 MICRO-SD-PUSH-PUSH-EXT-PIN, J4 Vertical Qwiic Connector, J9 MAGJACK-POE, U1 ESP32-WROVER-IE, U10 POE_PSU-DP990X, U11 MCP6021T, U12 AP7361C-33, U13 MCP6021T, U14 BP2G1+_POWER_SPLITTER, U15 USB251XB, U16 SN74AVC4T774PW, U17 URB2405YMD-15WR3, U2 CH340C, U3 XC6222B331MR-G, U4 U-BLOX_ZED-F9P, U5 U-BLOX_NEO-D9S-00B, U6 XC6222B331MR-G, U7 W5500, U8 LARA-R6001, U9 74LVC4066D_QUAD_BILATERAL_SWI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, Y1 25MHz, Y2 24MHz

Commit message: Add Route-Out gaps on panel
Other:
- board text added: "Controlled Impedance: JLC7628 Material: TG155 4-Layers Thickness: 1.6mm Outer Copper: 1oz Inner Copper: 0.5oz Finish: HASL Lead Free Red Solder Resist White Silkscreen"
- board text removed: "JLCPCB JLC-7628 Impedance Control 4-Layers Thickness: 1.6mm Outer Copper: 1oz Finish: HASL Lead Free Red Solder Resist White Silkscreen"
Changed lines of the file:
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@@
 <drawing>
 <settings>
-<setting alwaysvectorfont="yes"/>
+<setting alwaysvectorfont="no"/>
 <setting verticaltext="up"/>
 </settings>
@@
 <dimension x1="0" y1="101.6" x2="0" y2="0" x3="-8.89" y3="50.8" textsize="1.778" textratio="15" layer="47" dtype="vertical" unit="inch"/>
 <text x="213.36" y="0" size="1.778" layer="51" font="vector" ratio="15">Paul Clark</text>
-<text x="160.02" y="49.53" size="1.778" layer="51" font="vector" ratio="15" align="top-left">JLCPCB JLC-7628 Impedance Control
+<text x="160.02" y="49.53" size="1.778" layer="51" font="vector" ratio="15" align="top-left">Controlled Impedance: JLC7628
+Material: TG155
 4-Layers
 Thickness: 1.6mm
 Outer Copper: 1oz
+Inner Copper: 0.5oz
 Finish: HASL Lead Free
 Red Solder Resist

Commit message: Update Libraries, PROD_IDs etc.
Parts:
- U15: value USB251XB -> USB251XB_USB2514B; device USB251xB:QFN-36 -> SparkFun-IC-Special-Function:QFN-36
- U17: value URB2405YMD-15WR3 -> URB2405YMD
- U8: value LARA-R6001 -> LARA-R6001D
Changed lines of the file:
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@@
 <element name="U1" library="SparkFun-RF" package="ESP32-WROVER-E/IE" value="ESP32-WROVER-IE" x="92.71" y="43.18" smashed="yes" rot="R180">
 <attribute name="NAME" x="100.47" y="43.18" size="0.8128" layer="25" rot="R270" align="center"/>
+<attribute name="PROD_ID" value="IC-19265" x="92.71" y="43.18" size="1.778" layer="27" rot="R180" display="off"/>
 <attribute name="VALUE" x="99.2" y="43.18" size="0.8128" layer="27" rot="R270" align="center"/>
 </element>
@@
 <attribute name="REV" value="V01" x="185.42" y="1.27" size="1.778" layer="27" display="off"/>
 </element>
-<element name="U8" library="SparkFun-RF" package="LARA-LGA" value="LARA-R6001" x="132.08" y="72.39" smashed="yes" rot="R270">
+<element name="U8" library="SparkFun-RF" package="LARA-LGA" value="LARA-R6001D" x="132.08" y="72.39" smashed="yes" rot="R270">
 <attribute name="NAME" x="132.08" y="85.79" size="0.6096" layer="25" font="vector" ratio="20" align="bottom-center"/>
-<attribute name="VALUE" x="132.08" y="58.99" size="0.6096" layer="27" font="vector" ratio="20" rot="R180" align="bottom-center"/>
+<attribute name="PROD_ID" value="IC-16661" x="132.08" y="72.39" size="1.778" layer="27" rot="R270" display="off"/>
+<attribute name="VALUE" value="LARA-R6001D" x="132.08" y="58.99" size="0.6096" layer="27" font="vector" ratio="20" rot="R180" align="bottom-center"/>
 </element>
 <element name="C22" library="SparkFun-Capacitors" package="0603" value="2.2uF" x="62.23" y="36.195" smashed="yes">
@@
 <attribute name="VALUE" x="139.319" y="23.284" size="0.6096" layer="27" ratio="20" align="top-center"/>
 </element>
-<element name="U15" library="USB251xB" package="QFN-36" value="USB251XB" x="133.35" y="24.13" smashed="yes" rot="R270">
+<element name="U15" library="SparkFun-IC-Special-Function" package="QFN-36" value="USB251XB_USB2514B" x="133.35" y="24.13" smashed="yes" rot="R270">
 <attribute name="NAME" x="133.35" y="27.305" size="0.6096" layer="25" font="vector" ratio="20" align="bottom-center"/>
 <attribute name="PROD_ID" value="IC-15827" x="129.54" y="27.94" size="1.778" layer="27" ratio="15" rot="R270" display="off"/>
@@
 <element name="C86" library="SparkFun-Capacitors" package="PANASONIC_D" value="47UF" x="9.271" y="36.83" smashed="yes" rot="R270">
 <attribute name="NAME" x="12.7" y="36.83" size="0.6096" layer="25" font="vector" ratio="20" rot="R270" align="bottom-center"/>
+<attribute name="PROD_ID" value="CAP-10547" x="9.271" y="36.83" size="1.778" layer="27" rot="R270" display="off"/>
 <attribute name="VALUE" x="5.842" y="36.83" size="0.6096" layer="27" font="vector" ratio="20" rot="R270" align="top-center"/>
 </element>
-<element name="U17" library="SparkFun-IC-Power" package="URB_YMD-15WR3" value="URB2405YMD-15WR3" x="26.67" y="36.83" smashed="yes">
+<element name="U17" library="SparkFun-IC-Power" package="URB_YMD-15WR3" value="URB2405YMD" x="26.67" y="36.83" smashed="yes">
 <attribute name="NAME" x="13.97" y="49.53" size="1.27" layer="25" font="vector"/>
-<attribute name="PROD_ID" value="" x="26.67" y="36.83" size="1.778" layer="27" display="off"/>
-<attribute name="VALUE" x="13.97" y="22.86" size="1.27" layer="27" font="vector"/>
+<attribute name="PROD_ID" value="COMP-19263" x="26.67" y="36.83" size="1.778" layer="27" display="off"/>
+<attribute name="VALUE" value="URB2405YMD" x="13.97" y="22.86" size="1.27" layer="27" font="vector"/>
 </element>
 <element name="I2C1" library="SparkFun-Jumpers" package="SMT-JUMPER_3_NO_SILK" package3d_urn="urn:adsk.eagle:package:39285/1" value="JUMPER-SMT_3_NO_SILK" x="110.49" y="87.63" smashed="yes" rot="MR0">
