File: Hardware/RTK_Control.sch (EAGLE design)
At the start: 294 parts, among them J3 MICRO-SD-PUSH-PUSH-EXT-PIN, J4 Vertical Qwiic Connector, J9 MAGJACK-POE, U1 ESP32-WROVER-IE, U10 POE_PSU-DP990X, U11 MCP6021T, U12 AP7361C-33, U13 MCP6021T, U14 BP2G1+_POWER_SPLITTER, U15 USB251XB, U16 SN74AVC4T774PW, U17 URB2405YMD-15WR3, U2 CH340C, U3 XC6222B331MR-G, U4 U-BLOX_ZED-F9P, U5 U-BLOX_NEO-D9S-00B, U6 XC6222B331MR-G, U7 W5500, U8 LARA-R6001, U9 74LVC4066D_QUAD_BILATERAL_SWI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, Y1 25MHz, Y2 24MHz

Commit message: Almost routed
Connections:
- net ESP13/LARA_TXDI: now also U16.B3; no longer U16.B1
- net ESP34/LARA_NI: now also U16.B1; no longer U16.B3
- net GND: now also U16.DIR3; no longer U16.DIR1
- net LARA_18_NI: now also U16.A1; no longer U16.A3
- net LARA_18_TXDI: now also U16.A3; no longer U16.A1
- net VCCIO: now also U16.DIR1; no longer U16.DIR3
Changed lines of the file:
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@@
-</segment>
-<segment>
-<pinref part="U16" gate="G$1" pin="DIR1"/>
-<wire x1="284.48" y1="254" x2="281.94" y2="254" width="0.1524" layer="91"/>
-<pinref part="GND108" gate="1" pin="GND"/>
-<wire x1="281.94" y1="254" x2="281.94" y2="231.14" width="0.1524" layer="91"/>
 </segment>
 <segment>
@@
 <pinref part="Q4" gate="G1" pin="E"/>
 <wire x1="388.62" y1="99.06" x2="388.62" y2="101.6" width="0.1524" layer="91"/>
+</segment>
+<segment>
+<pinref part="U16" gate="G$1" pin="DIR3"/>
+<wire x1="284.48" y1="238.76" x2="281.94" y2="238.76" width="0.1524" layer="91"/>
+<pinref part="GND108" gate="1" pin="GND"/>
+<wire x1="281.94" y1="238.76" x2="281.94" y2="231.14" width="0.1524" layer="91"/>
 </segment>
 </net>
@@
 </segment>
 <segment>
+<pinref part="U16" gate="G$1" pin="DIR1"/>
+<wire x1="284.48" y1="254" x2="279.4" y2="254" width="0.1524" layer="91"/>
+<pinref part="SUPPLY75" gate="G$1" pin="VCCIO"/>
+<wire x1="279.4" y1="254" x2="279.4" y2="256.54" width="0.1524" layer="91"/>
 <pinref part="U16" gate="G$1" pin="DIR2"/>
 <wire x1="284.48" y1="251.46" x2="279.4" y2="251.46" width="0.1524" layer="91"/>
-<pinref part="SUPPLY75" gate="G$1" pin="VCCIO"/>
-<wire x1="279.4" y1="251.46" x2="279.4" y2="256.54" width="0.1524" layer="91"/>
-<pinref part="U16" gate="G$1" pin="DIR3"/>
-<wire x1="284.48" y1="238.76" x2="279.4" y2="238.76" width="0.1524" layer="91"/>
-<wire x1="279.4" y1="238.76" x2="279.4" y2="241.3" width="0.1524" layer="91"/>
+<wire x1="279.4" y1="251.46" x2="279.4" y2="254" width="0.1524" layer="91"/>
+<junction x="279.4" y="254"/>
+<pinref part="U16" gate="G$1" pin="DIR4"/>
+<wire x1="284.48" y1="236.22" x2="279.4" y2="236.22" width="0.1524" layer="91"/>
+<wire x1="279.4" y1="236.22" x2="279.4" y2="241.3" width="0.1524" layer="91"/>
 <junction x="279.4" y="251.46"/>
-<pinref part="U16" gate="G$1" pin="DIR4"/>
+<pinref part="U16" gate="G$1" pin="A4"/>
 <wire x1="279.4" y1="241.3" x2="279.4" y2="251.46" width="0.1524" layer="91"/>
-<wire x1="284.48" y1="236.22" x2="279.4" y2="236.22" width="0.1524" layer="91"/>
-<wire x1="279.4" y1="236.22" x2="279.4" y2="238.76" width="0.1524" layer="91"/>
-<junction x="279.4" y="238.76"/>
-<pinref part="U16" gate="G$1" pin="A4"/>
 <wire x1="284.48" y1="241.3" x2="279.4" y2="241.3" width="0.1524" layer="91"/>
 <junction x="279.4" y="241.3"/>
@@
 </segment>
 <segment>
-<pinref part="U16" gate="G$1" pin="A1"/>
-<wire x1="284.48" y1="248.92" x2="276.86" y2="248.92" width="0.1524" layer="91"/>
-<label x="276.86" y="248.92" size="1.27" layer="95" rot="R180" xref="yes"/>
+<label x="276.86" y="243.84" size="1.27" layer="95" rot="R180" xref="yes"/>
+<pinref part="U16" gate="G$1" pin="A3"/>
+<wire x1="284.48" y1="243.84" x2="276.86" y2="243.84" width="0.1524" layer="91"/>
 </segment>
 </net>
@@
 </segment>
 <segment>
+<label x="276.86" y="246.38" size="1.27" layer="95" rot="R180" xref="yes"/>
 <pinref part="U16" gate="G$1" pin="A2"/>
-<wire x1="284.48" y1="246.38" x2="276.86" y2="246.38" width="0.1524" layer="91"/>
-<label x="276.86" y="246.38" size="1.27" layer="95" rot="R180" xref="yes"/>
+<wire x1="276.86" y1="246.38" x2="284.48" y2="246.38" width="0.1524" layer="91"/>
 </segment>
 </net>
 <net name="ESP13/LARA_TXDI" class="0">
 <segment>
-<pinref part="U16" gate="G$1" pin="B1"/>
-<wire x1="307.34" y1="248.92" x2="309.88" y2="248.92" width="0.1524" layer="91"/>
-<label x="309.88" y="248.92" size="1.27" layer="95" xref="yes"/>
+<label x="309.88" y="243.84" size="1.27" layer="95" xref="yes"/>
+<pinref part="U16" gate="G$1" pin="B3"/>
+<wire x1="307.34" y1="243.84" x2="309.88" y2="243.84" width="0.1524" layer="91"/>
 </segment>
 </net>
@@
 </segment>
 <segment>
-<pinref part="U16" gate="G$1" pin="A3"/>
-<wire x1="284.48" y1="243.84" x2="276.86" y2="243.84" width="0.1524" layer="91"/>
-<label x="276.86" y="243.84" size="1.27" layer="95" rot="R180" xref="yes"/>
+<label x="276.86" y="248.92" size="1.27" layer="95" rot="R180" xref="yes"/>
+<pinref part="U16" gate="G$1" pin="A1"/>
+<wire x1="284.48" y1="248.92" x2="276.86" y2="248.92" width="0.1524" layer="91"/>
 </segment>
 </net>
 <net name="ESP34/LARA_NI" class="0">
 <segment>
-<pinref part="U16" gate="G$1" pin="B3"/>
-<wire x1="307.34" y1="243.84" x2="309.88" y2="243.84" width="0.1524" layer="91"/>
-<label x="309.88" y="243.84" size="1.27" layer="95" xref="yes"/>
-</segment>
-</net>
+<label x="309.88" y="248.92" size="1.27" layer="95" xref="yes"/>
+<pinref part="U16" gate="G$1" pin="B1"/>
+<wire x1="307.34" y1="248.92" x2="309.88" y2="248.92" width="0.1524" layer="91"/>
+</segment>
+</net>

Commit message: Ready for Proto Review
Connections:
- net N$26 renamed NEO_TXO
- net N$31 renamed NEO_RXI
- net N$67 renamed VIN2+
Changed lines of the file:
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@@
 </segment>
 </net>
-<net name="N$67" class="0">
+<net name="VIN2+" class="0">
 <segment>
 <pinref part="U17" gate="U1" pin="VIN+"/>
@@
 </segment>
 </net>
-<net name="N$26" class="0">
+<net name="NEO_TXO" class="0">
 <segment>
 <pinref part="U5" gate="U1" pin="TXD1/POCI"/>
@@
 </segment>
 </net>
-<net name="N$31" class="0">
+<net name="NEO_RXI" class="0">
 <segment>
 <pinref part="U5" gate="U1" pin="RXD1/PICO"/>

Commit message: Update Libraries, PROD_IDs etc.
Parts:
- U1: device SparkFun-RF:ESP32-WROVER-E/IE -> SparkFun-RF:ESP32-WROVER-E/IE_IE-N16R8
- U15: value USB251XB -> USB251XB_USB2514B; device USB251xB:USB251XB -> SparkFun-IC-Special-Function:USB251XB_USB2514B
- U17: value URB2405YMD-15WR3 -> URB2405YMD
- U8: value LARA-R6001 -> LARA-R6001D; device SparkFun-RF:LARA-R6001 -> SparkFun-RF:LARA-R6_R6001D_GLOBAL_DATA-ONLY
Other:
- note added: "USB2513, or USB2514 can be used"
- note removed: "Any USB2512*, USB2513, or USB2514 can be used USB2513 or higher required for NEO variant"
Changed lines of the file:
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@@
 <part name="FD3" library="SparkFun-Aesthetics" deviceset="FIDUCIAL" device="1X2"/>
 <part name="FD4" library="SparkFun-Aesthetics" deviceset="FIDUCIAL" device="1X2"/>
-<part name="U1" library="SparkFun-RF" deviceset="ESP32-WROVER-E/IE" device="" value="ESP32-WROVER-IE"/>
+<part name="U1" library="SparkFun-RF" deviceset="ESP32-WROVER-E/IE" device="_IE-N16R8" value="ESP32-WROVER-IE"/>
 <part name="GND1" library="SparkFun-PowerSymbols" deviceset="GND" device=""/>
 <part name="SUPPLY1" library="SparkFun-PowerSymbols" deviceset="3.3V" device=""/>
@@
 <attribute name="REV" value="V01"/>
 </part>
-<part name="U8" library="SparkFun-RF" deviceset="LARA-R6001" device="" value="LARA-R6001"/>
+<part name="U8" library="SparkFun-RF" deviceset="LARA-R6" device="_R6001D_GLOBAL_DATA-ONLY" value="LARA-R6001D"/>
 <part name="GND25" library="SparkFun-PowerSymbols" deviceset="GND" device=""/>
 <part name="C22" library="SparkFun-Capacitors" deviceset="2.2UF" device="-0603-10V-20%" value="2.2uF"/>
@@
 <part name="R12" library="SparkFun-Resistors" deviceset="12KOHM" device="-0603-1/10W-1%" value="12k"/>
 <part name="Y2" library="SparkFun-Clocks" deviceset="CRYSTAL-24MHZ" device="-SMD-2.0X1.6MM" value="24MHz"/>
-<part name="U15" library="USB251xB" deviceset="USB251XB" device=""/>
+<part name="U15" library="SparkFun-IC-Special-Function" deviceset="USB251XB" device="_USB2514B"/>
 <part name="R13" library="SparkFun-Resistors" deviceset="1MOHM" device="-0603-1/4W-5%" value="1M"/>
 <part name="C63" library="SparkFun-Capacitors" deviceset="18PF" device="-0603-50V-5%" value="18pF"/>
@@
 <part name="GND128" library="SparkFun-PowerSymbols" deviceset="GND" device=""/>
 <part name="C86" library="SparkFun-Capacitors" deviceset="47UF-POLAR" device="-PANASONIC_D-50V-20%" value="47UF"/>
-<part name="U17" library="SparkFun-IC-Power" deviceset="URB_YMD-15WR3" device="__URB2405YMD-15WR3" value="URB2405YMD-15WR3"/>
+<part name="U17" library="SparkFun-IC-Power" deviceset="URB_YMD-15WR3" device="__URB2405YMD-15WR3" value="URB2405YMD"/>
 <part name="I2C1" library="SparkFun-Jumpers" deviceset="JUMPER-SMT_3_NO" device="_SILK" package3d_urn="urn:adsk.eagle:package:39285/1"/>
 <part name="R71" library="SparkFun-Resistors" deviceset="2.2KOHM" device="-0603-1/10W-1%" value="2.2k"/>
@@
 <text x="326.39" y="187.96" size="1.778" layer="97" font="vector">90Ω</text>
 <text x="279.4" y="81.28" size="1.778" layer="97" font="vector" align="center">7-bit unshifted I²C address: 0x2C</text>
-<text x="279.4" y="76.2" size="1.27" layer="97" font="vector" align="center">Any USB2512*, USB2513, or USB2514 can be used
-USB2513 or higher required for NEO variant</text>
+<text x="279.4" y="78.74" size="1.27" layer="97" font="vector" align="center">USB2513, or USB2514 can be used</text>
 <text x="149.86" y="152.4" size="2.54" layer="94" font="vector" align="top-left">USB Hub</text>
 <wire x1="180.34" y1="60.96" x2="330.2" y2="60.96" width="0.1524" layer="97" style="longdash"/>
