File: Hardware/SparkFun_RTK_EVK.sch (EAGLE design)
At the start: 311 parts, among them J3 MICRO-SD-PUSH-PUSH-EXT-PIN, J4 Vertical Qwiic Connector, J9 MAGJACK-POE, Q5 310mA/60V/1.6Ω, Q6 310mA/60V/1.6Ω, U1 ESP32-WROVER-IE, U10 POE_PSU-DP990X, U11 MCP6021T, U12 AP7361C-33, U13 MCP6021T, U14 BP2G1+_POWER_SPLITTER, U15 USB251XB_USB2514B, U16 SN74AVC4T774PW, U17 URB2405YMD, U18 74HC1G04, U2 CH340C, U3 XC6222B331MR-G, U4 U-BLOX_ZED-F9P, U5 U-BLOX_NEO-D9S-00B, U6 XC6222B331MR-G, U7 W5500, U8 LARA-R6001D, U9 74LVC4066D_QUAD_BILATERAL_SWI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, Y1 25MHz, Y2 24MHz

Commit message: v11 PCB
Parts:
- removed LARA_ON: TEST-POINTPOGO_PTH, SparkFun-Connectors:TEST-POINTPOGO_PTH
- removed RX-TX, TX-RX: JUMPER-COMBO_2_NC_TRACE, SparkFun-Jumpers:JUMPER-COMBO_2_NC_TRACE
- added NEO_RX, NEO_TX, ZED_RXI, ZED_TXO: TEST-POINTPOGO_PTH, SparkFun-Connectors:TEST-POINTPOGO_PTH
Connections:
- net ESP5/LARA_ON renamed ESP5/TP
- removed net ESP25/TP: D20.1, J13.1, R6.2, TP.1, U1.DAC1/IOA25
- removed net ESP33/!ETH_INT!: ETH_INT.1, U1.XTAL_N/IOA33, U7.!INT!
- removed net LARA_ON: LARA_ON.1, U16.B4, U9.3Z
- removed net ZED_RXI: RX-TX.2, U4.RX/MOSI
- removed net ZED_TXO: TX-RX.1, U4.TX/MISO
- new net ESP25/ZED_TXO: U1.DAC1/IOA25, U4.TX/MISO, ZED_TXO.1
- new net ESP33/ZED_RXI: U1.XTAL_N/IOA33, U4.RX/MOSI, ZED_RXI.1
- new net ESP39/!ETH_INT!: ETH_INT.1, U1.SENSOR_VN/IA39, U7.!INT!
- new net ZED_TP: D20.1, J13.1, R6.2, TP.1, U9.3Z
- net NEO_RXI: now also NEO_RX.1; no longer TX-RX.2
- net NEO_TXO: now also NEO_TX.1; no longer RX-TX.1
Other:
- note added: "v11"
- note removed: "v10"

Commit message: Final tweaks
Parts:
- I2C: value JUMPER-SMT_3_2-NC_TRACE_SILK -> JUMPER-SMT_3_NO_SILK; device SparkFun-Jumpers:JUMPER-SMT_3_2-NC_TRACE_SILK -> SparkFun-Jumpers:JUMPER-SMT_3_NO_SILK
Other:
- note removed: "Open jumpers to disable pull-ups"
Changed lines of the file:
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@@
 <part name="SUPPLY37" library="SparkFun-PowerSymbols" deviceset="3.3V" device=""/>
 <part name="SUPPLY41" library="SparkFun-PowerSymbols" deviceset="3.3V" device=""/>
-<part name="I2C" library="SparkFun-Jumpers" deviceset="JUMPER-SMT_3_2-NC_TRACE" device="_SILK" package3d_urn="urn:adsk.eagle:package:39289/1"/>
+<part name="I2C" library="SparkFun-Jumpers" deviceset="JUMPER-SMT_3_NO" device="_SILK" package3d_urn="urn:adsk.eagle:package:39285/1"/>
 <part name="R16" library="SparkFun-Resistors" deviceset="2.2KOHM" device="-0603-1/10W-1%" value="2.2k"/>
 <part name="R19" library="SparkFun-Resistors" deviceset="2.2KOHM" device="-0603-1/10W-1%" value="2.2k"/>
@@
 <wire x1="345.44" y1="46.99" x2="391.16" y2="46.99" width="0.2032" layer="97"/>
 <wire x1="345.44" y1="44.45" x2="391.16" y2="44.45" width="0.2032" layer="97"/>
-<text x="309.88" y="74.93" size="1.27" layer="97" font="vector" rot="R180" align="bottom-center">Open jumpers to
-disable pull-ups</text>
+<text x="309.88" y="74.93" size="1.27" layer="97" font="vector" rot="R180" align="bottom-center">Close jumpers to
+enable pull-ups</text>
 <text x="107.95" y="185.42" size="1.27" layer="97" font="vector" align="bottom-center">Open jumper to isolate shield</text>
 <text x="268.986" y="266.954" size="1.778" layer="97" font="vector">Vin Max: 6.0V
